File: hardware/Hauptplatine/Hauptplatine_v3.3cy_logic_minimal_150x90.kicad_pcb (KiCad board)
At the start: 2 copper layers, 150 x 90 mm, 29 parts, among them J1 230V IN L/N/PE, J2 REED OFFEN, J3 REED GEKIPPT, J4 RS485 5V/GND/A/B, J5 MOTOR N/PE/AUF/AB, J6 28BYJ-48 OBEN, J7 28BYJ-48 UNTEN, K1 Finder 40.52.9.005.0000 AUF, K2 Finder 40.52.9.005.0000 AB, Q1 BC337 AUF, Q2 BC337 AB, U1 ESP32-S3 DevKitC-1 headers, U2 AMS1117-3.3, U3 MAX3485, U4 ULN2003A OBEN, U5 ULN2003A UNTEN

Commit message: PCB v3.3cy: reconnect AC_L after F2 relocation
Routing:
- net /AC_L: track 64.7 -> 73.7 mm
Changed lines of the file:
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@@
 	(segment
 		(start 36 40.8)
-		(end 30 40.8)
+		(end 30 54.6)
 		(width 2)
 		(layer "F.Cu")
