File: hardware/Sensorplatine/Sensorplatine_v1.0_routing_draft_50x50.kicad_pcb (KiCad board)
At the start: 2 copper layers, 50 x 50 mm, 11 parts, among them J1 5V/GND/A/B, M1 HLK-LD2450, U1 STM32G031K8T6, U2 BME280 - LANDPATTERN TODO, U3 SCD41 - LANDPATTERN TODO, U4 SGP40 - LANDPATTERN TODO, U5 VEML7700 - LANDPATTERN TODO, U7 MAX3485, U8 T5848 - LANDPATTERN TODO, U9 AP2112K-3.3

Commit message: hardware: route I2C LD2450 I2S and SWD trunks
Parts:
- added J2: SWD, Sensorplatine:SWD_1x05, F.Cu at (145.0, 146.0)
- added J3: LD2450 temporary interface, Sensorplatine:LD2450_IF, F.Cu at (125.0, 118.0)
- added TP_I2C: I2C trunk to sensor zone, Sensorplatine:I2C_TEMP_TERMINALS, F.Cu at (125.0, 127.0)
- added TP_I2S: I2S trunk to microphone zone, Sensorplatine:I2S_TEMP_TERMINALS, F.Cu at (143.0, 137.0)
Connections:
- U1 pad 1: (no net) -> I2C_SDA
- U1 pad 10: (no net) -> LD2450_TX
- U1 pad 11: (no net) -> I2S_WS
- U1 pad 12: (no net) -> I2S_CK
- U1 pad 14: (no net) -> I2S_SD
- U1 pad 24: (no net) -> SWDIO
- U1 pad 25: (no net) -> SWCLK
- U1 pad 28: (no net) -> I2C_SCL
- U1 pad 6: (no net) -> NRST
- U1 pad 9: (no net) -> LD2450_RX
Routing:
- net GND: track 21.9 -> 81.3 mm
- net +3V3: track 14.3 -> 51.9 mm
- net NRST: track 0.00 -> 26.6 mm
- net +5V: track 8.38 -> 32.1 mm
- net LD2450_RX: track 0.00 -> 23.3 mm
- net LD2450_TX: track 0.00 -> 22.5 mm
- net SWCLK: track 0.00 -> 21.7 mm
- net SWDIO: track 0.00 -> 19.8 mm
- net I2S_SD: track 0.00 -> 19.3 mm
- net I2S_CK: track 0.00 -> 18.8 mm
- net I2S_WS: track 0.00 -> 17.3 mm
- net I2C_SDA: track 0.00 -> 6.26 mm
- net I2C_SCL: track 0.00 -> 4.91 mm
Other:
- board text added: "I2C routed to sensor zone"
- board text added: "I2S routed to microphone zone"
- board text added: "LD2450 UART + 5V/GND routed to module interface"
- board text added: "SWD fully routed"
Changed lines of the file:
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@@
   (net 7 "RS485_RX")
   (net 8 "RS485_DE")
+  (net 9 "I2C_SDA")
+  (net 10 "I2C_SCL")
+  (net 11 "LD2450_TX")
+  (net 12 "LD2450_RX")
+  (net 13 "I2S_WS")
+  (net 14 "I2S_CK")
+  (net 15 "I2S_SD")
+  (net 16 "SWDIO")
+  (net 17 "SWCLK")
+  (net 18 "NRST")
   (gr_rect (start 100 100) (end 150 150)
     (stroke (width 0.2) (type default)) (fill none) (layer "Edge.Cuts"))
@@
     (fp_text value "STM32G031K8T6" (at 0 5) (layer "F.Fab")
       (effects (font (size 0.8 0.8) (thickness 0.12))))
-    (pad "1" smd rect (at -4.15 -3.5) (size 1.2 0.45) (layers "F.Cu" "F.Paste" "F.Mask"))
+    (pad "1" smd rect (at -4.15 -3.5) (size 1.2 0.45) (layers "F.Cu" "F.Paste" "F.Mask") (net 9 "I2C_SDA"))
     (pad "2" smd rect (at -4.15 -2.5) (size 1.2 0.45) (layers "F.Cu" "F.Paste" "F.Mask"))
     (pad "3" smd rect (at -4.15 -1.5) (size 1.2 0.45) (layers "F.Cu" "F.Paste" "F.Mask"))
     (pad "4" smd rect (at -4.15 -0.5) (size 1.2 0.45) (layers "F.Cu" "F.Paste" "F.Mask") (net 3 "+3V3"))
     (pad "5" smd rect (at -4.15 0.5) (size 1.2 0.45) (layers "F.Cu" "F.Paste" "F.Mask") (net 1 "GND"))
-    (pad "6" smd rect (at -4.15 1.5) (size 1.2 0.45) (layers "F.Cu" "F.Paste" "F.Mask"))
+    (pad "6" smd rect (at -4.15 1.5) (size 1.2 0.45) (layers "F.Cu" "F.Paste" "F.Mask") (net 18 "NRST"))
     (pad "7" smd rect (at -4.15 2.5) (size 1.2 0.45) (layers "F.Cu" "F.Paste" "F.Mask"))
     (pad "8" smd rect (at -4.15 3.5) (size 1.2 0.45) (layers "F.Cu" "F.Paste" "F.Mask"))
-    (pad "9" smd rect (at -3.5 4.15) (size 0.45 1.2) (layers "F.Cu" "F.Paste" "F.Mask"))
-    (pad "10" smd rect (at -2.5 4.15) (size 0.45 1.2) (layers "F.Cu" "F.Paste" "F.Mask"))
-    (pad "11" smd rect (at -1.5 4.15) (size 0.45 1.2) (layers "F.Cu" "F.Paste" "F.Mask"))
-    (pad "12" smd rect (at -0.5 4.15) (size 0.45 1.2) (layers "F.Cu" "F.Paste" "F.Mask"))
+    (pad "9" smd rect (at -3.5 4.15) (size 0.45 1.2) (layers "F.Cu" "F.Paste" "F.Mask") (net 12 "LD2450_RX"))
+    (pad "10" smd rect (at -2.5 4.15) (size 0.45 1.2) (layers "F.Cu" "F.Paste" "F.Mask") (net 11 "LD2450_TX"))
+    (pad "11" smd rect (at -1.5 4.15) (size 0.45 1.2) (layers "F.Cu" "F.Paste" "F.Mask") (net 13 "I2S_WS"))
+    (pad "12" smd rect (at -0.5 4.15) (size 0.45 1.2) (layers "F.Cu" "F.Paste" "F.Mask") (net 14 "I2S_CK"))
     (pad "13" smd rect (at 0.5 4.15) (size 0.45 1.2) (layers "F.Cu" "F.Paste" "F.Mask"))
-    (pad "14" smd rect (at 1.5 4.15) (size 0.45 1.2) (layers "F.Cu" "F.Paste" "F.Mask"))
+    (pad "14" smd rect (at 1.5 4.15) (size 0.45 1.2) (layers "F.Cu" "F.Paste" "F.Mask") (net 15 "I2S_SD"))
     (pad "15" smd rect (at 2.5 4.15) (size 0.45 1.2) (layers "F.Cu" "F.Paste" "F.Mask"))
     (pad "16" smd rect (at 3.5 4.15) (size 0.45 1.2) (layers "F.Cu" "F.Paste" "F.Mask") (net 8 "RS485_DE"))
@@
     (pad "22" smd rect (at 4.15 -1.5) (size 1.2 0.45) (layers "F.Cu" "F.Paste" "F.Mask"))
     (pad "23" smd rect (at 4.15 -2.5) (size 1.2 0.45) (layers "F.Cu" "F.Paste" "F.Mask"))
-    (pad "24" smd rect (at 4.15 -3.5) (size 1.2 0.45) (layers "F.Cu" "F.Paste" "F.Mask"))
-    (pad "25" smd rect (at 3.5 -4.15) (size 0.45 1.2) (layers "F.Cu" "F.Paste" "F.Mask"))
+    (pad "24" smd rect (at 4.15 -3.5) (size 1.2 0.45) (layers "F.Cu" "F.Paste" "F.Mask") (net 16 "SWDIO"))
+    (pad "25" smd rect (at 3.5 -4.15) (size 0.45 1.2) (layers "F.Cu" "F.Paste" "F.Mask") (net 17 "SWCLK"))
     (pad "26" smd rect (at 2.5 -4.15) (size 0.45 1.2) (layers "F.Cu" "F.Paste" "F.Mask"))
     (pad "27" smd rect (at 1.5 -4.15) (size 0.45 1.2) (layers "F.Cu" "F.Paste" "F.Mask") (net 7 "RS485_RX"))
-    (pad "28" smd rect (at 0.5 -4.15) (size 0.45 1.2) (layers "F.Cu" "F.Paste" "F.Mask"))
+    (pad "28" smd rect (at 0.5 -4.15) (size 0.45 1.2) (layers "F.Cu" "F.Paste" "F.Mask") (net 10 "I2C_SCL"))
     (pad "29" smd rect (at -0.5 -4.15) (size 0.45 1.2) (layers "F.Cu" "F.Paste" "F.Mask"))
     (pad "30" smd rect (at -1.5 -4.15) (size 0.45 1.2) (layers "F.Cu" "F.Paste" "F.Mask"))
@@
     (fp_text value "T5848 - LANDPATTERN TODO" (at 0 2.5) (layer "F.Fab")
       (effects (font (size 0.6 0.6) (thickness 0.1))))
+  )
+  (footprint "Sensorplatine:I2C_TEMP_TERMINALS" (layer "F.Cu") (at 125 127)
+    (fp_text reference "TP_I2C" (at 0 -2.5) (layer "F.SilkS") (effects (font (size 0.7 0.7) (thickness 0.1))))
+    (fp_text value "I2C trunk to sensor zone" (at 0 2.5) (layer "F.Fab") (effects (font (size 0.6 0.6) (thickness 0.1))))
+    (pad "1" thru_hole circle (at -1.27 0) (size 1.5 1.5) (drill 0.7) (layers "*.Cu" "*.Mask") (net 9 "I2C_SDA"))
+    (pad "2" thru_hole circle (at 1.27 0) (size 1.5 1.5) (drill 0.7) (layers "*.Cu" "*.Mask") (net 10 "I2C_SCL"))
+  )
+  (footprint "Sensorplatine:LD2450_IF" (layer "F.Cu") (at 125 118)
+    (fp_text reference "J3" (at 0 -2.5) (layer "F.SilkS") (effects (font (size 0.7 0.7) (thickness 0.1))))
+    (fp_text value "LD2450 temporary interface" (at 0 2.5) (layer "F.Fab") (effects (font (size 0.6 0.6) (thickness 0.1))))
+    (pad "1" thru_hole circle (at -3.81 0) (size 1.6 1.6) (drill 0.8) (layers "*.Cu" "*.Mask") (net 2 "+5V"))
+    (pad "2" thru_hole circle (at -1.27 0) (size 1.6 1.6) (drill 0.8) (layers "*.Cu" "*.Mask") (net 1 "GND"))
+    (pad "3" thru_hole circle (at 1.27 0) (size 1.6 1.6) (drill 0.8) (layers "*.Cu" "*.Mask") (net 11 "LD2450_TX"))
+    (pad "4" thru_hole circle (at 3.81 0) (size 1.6 1.6) (drill 0.8) (layers "*.Cu" "*.Mask") (net 12 "LD2450_RX"))
+  )
+  (footprint "Sensorplatine:I2S_TEMP_TERMINALS" (layer "F.Cu") (at 143 137)
+    (fp_text reference "TP_I2S" (at 0 -2.5) (layer "F.SilkS") (effects (font (size 0.7 0.7) (thickness 0.1))))
+    (fp_text value "I2S trunk to microphone zone" (at 0 2.5) (layer "F.Fab") (effects (font (size 0.6 0.6) (thickness 0.1))))
+    (pad "1" thru_hole circle (at -2.54 0) (size 1.5 1.5) (drill 0.7) (layers "*.Cu" "*.Mask") (net 13 "I2S_WS"))
+    (pad "2" thru_hole circle (at 0 0) (size 1.5 1.5) (drill 0.7) (layers "*.Cu" "*.Mask") (net 14 "I2S_CK"))
+    (pad "3" thru_hole circle (at 2.54 0) (size 1.5 1.5) (drill 0.7) (layers "*.Cu" "*.Mask") (net 15 "I2S_SD"))
+  )
+  (footprint "Sensorplatine:SWD_1x05" (layer "F.Cu") (at 145 146 90)
+    (fp_text reference "J2" (at 0 -2.5 90) (layer "F.SilkS") (effects (font (size 0.8 0.8) (thickness 0.12))))
+    (fp_text value "SWD" (at 0 2.5 90) (layer "F.Fab") (effects (font (size 0.7 0.7) (thickness 0.1))))
+    (pad "1" thru_hole circle (at -5.08 0 90) (size 1.7 1.7) (drill 0.8) (layers "*.Cu" "*.Mask") (net 3 "+3V3"))
+    (pad "2" thru_hole circle (at -2.54 0 90) (size 1.7 1.7) (drill 0.8) (layers "*.Cu" "*.Mask") (net 16 "SWDIO"))
+    (pad "3" thru_hole circle (at 0 0 90) (size 1.7 1.7) (drill 0.8) (layers "*.Cu" "*.Mask") (net 17 "SWCLK"))
+    (pad "4" thru_hole circle (at 2.54 0 90) (size 1.7 1.7) (drill 0.8) (layers "*.Cu" "*.Mask") (net 18 "NRST"))
+    (pad "5" thru_hole circle (at 5.08 0 90) (size 1.7 1.7) (drill 0.8) (layers "*.Cu" "*.Mask") (net 1 "GND"))
   )
   (segment (start 104 139.25) (end 108.5 139.25) (width 0.6) (layer "F.Cu") (net 2))
@@
   (segment (start 118.2 137.905) (end 120.85 136.5) (width 0.5) (layer "B.Cu") (net 1))
   (segment (start 110 144.05) (end 111 139.95) (width 0.4) (layer "B.Cu") (net 1))
+  (segment (start 120.85 132.5) (end 121.5 131.85) (width 0.25) (layer "F.Cu") (net 9))
+  (segment (start 121.5 131.85) (end 123.73 127) (width 0.25) (layer "F.Cu") (net 9))
+  (segment (start 125.5 131.85) (end 126.27 127) (width 0.25) (layer "F.Cu") (net 10))
+  (segment (start 122.5 140.15) (end 126.27 118) (width 0.25) (layer "B.Cu") (net 11))
+  (segment (start 121.5 140.15) (end 128.81 118) (width 0.25) (layer "B.Cu") (net 12))
+  (segment (start 121.19 118) (end 112.2 139.95) (width 0.45) (layer "B.Cu") (net 2))
+  (segment (start 123.73 118) (end 111 139.95) (width 0.45) (layer "B.Cu") (net 1))
+  (segment (start 123.5 140.15) (end 140.46 137) (width 0.25) (layer "F.Cu") (net 13))
+  (segment (start 124.5 140.15) (end 143 137) (width 0.25) (layer "F.Cu") (net 14))
+  (segment (start 126.5 140.15) (end 145.54 137) (width 0.25) (layer "F.Cu") (net 15))
+  (segment (start 129.15 132.5) (end 142.46 143.46) (width 0.25) (layer "B.Cu") (net 16))
+  (segment (start 142.46 143.46) (end 145 143.46) (width 0.25) (layer "B.Cu") (net 16))
+  (segment (start 128.5 131.85) (end 145 146) (width 0.25) (layer "F.Cu") (net 17))
+  (segment (start 120.85 137.5) (end 145 148.54) (width 0.25) (layer "B.Cu") (net 18))
+  (segment (start 109.8 138.05) (end 145 151.08) (width 0.4) (layer "B.Cu") (net 3))
+  (segment (start 111 139.95) (end 145 140.92) (width 0.45) (layer "B.Cu") (net 1))
+  (gr_text "I2C routed to sensor zone" (at 126 129) (layer "Dwgs.User")
+    (effects (font (size 0.65 0.65) (thickness 0.1))))
+  (gr_text "LD2450 UART + 5V/GND routed to module interface" (at 125 120.5) (layer "Dwgs.User")
+    (effects (font (size 0.65 0.65) (thickness 0.1))))
+  (gr_text "I2S routed to microphone zone" (at 141.5 134.5) (layer "Dwgs.User")
+    (effects (font (size 0.65 0.65) (thickness 0.1))))
+  (gr_text "SWD fully routed" (at 141.5 142) (layer "Dwgs.User")
+    (effects (font (size 0.65 0.65) (thickness 0.1))))
   (gr_text "CORE ROUTED: POWER + RS485" (at 118 146.5)
     (layer "Dwgs.User")
